Commit message: WIP Phase 1: move non-Phase-1 code to 'extra', rebuild SLAM/Nav2/delivery/docking
- Web dashboard, battery simulator, demo scripts moved to branch 'extra'
- World: solid table bases (visible to 2D LiDAR), dock relocated to east wall
- Robot: frictionless raised casters + sphere wheel contacts (accurate odometry)
- SLAM: slam_toolbox params, world-anchored map saver, autonomous mapping tour,
  new map built by SLAM in simulation
- Nav2: Jazzy params (Smac 2D planner, MPPI, 0.38 m footprint, AMCL initial
  pose, collision monitor, opennav docking server with home_dock)
- Delivery task manager: FIFO queue driving NavigateToPose (kitchen -> table)
- Docking controller: idle/manual/low-battery triggers via DockRobot/UndockRobot

Still to verify end-to-end: full system launch (deliveries + docking).

Co-Authored-By: Claude Opus 5.5 <noreply@anthropic.com>
Claude-Session: https://claude.ai/code/session_01HAZSW8R7SG4hPQGxKVJYa9

File: ros2_ws/src/cstam_gazebo/urdf/cstam_robot.urdf.xacro (robot description, xacro)
@@ -59,8 +59,10 @@
       <material name="metallic_dark"/>
     </visual>
-    <collision>
-      <origin xyz="0 0 0" rpy="1.5707963 0 0"/>
-      <geometry>
-        <cylinder radius="0.09" length="0.045"/>
+    <!-- Sphere collision: a single, well-defined contact point under the
+         axle keeps wheel odometry consistent with the real motion -->
+    <collision>
+      <origin xyz="0 0 0" rpy="0 0 0"/>
+      <geometry>
+        <sphere radius="0.09"/>
       </geometry>
     </collision>
@@ -85,8 +87,10 @@
       <material name="metallic_dark"/>
     </visual>
-    <collision>
-      <origin xyz="0 0 0" rpy="1.5707963 0 0"/>
-      <geometry>
-        <cylinder radius="0.09" length="0.045"/>
+    <!-- Sphere collision: a single, well-defined contact point under the
+         axle keeps wheel odometry consistent with the real motion -->
+    <collision>
+      <origin xyz="0 0 0" rpy="0 0 0"/>
+      <geometry>
+        <sphere radius="0.09"/>
       </geometry>
     </collision>
@@ -102,12 +106,13 @@
     <axis xyz="0 1 0"/>
   </joint>
-  <!-- Front Passive Caster -->
+  <!-- Front Passive Caster (5 mm above the floor so the drive wheels always
+       carry the robot's weight and never lose traction) -->
   <link name="caster_front">
     <visual>
-      <geometry><sphere radius="0.045"/></geometry>
-      <material name="metallic_dark"/>
-    </visual>
-    <collision>
-      <geometry><sphere radius="0.045"/></geometry>
+      <geometry><sphere radius="0.040"/></geometry>
+      <material name="metallic_dark"/>
+    </visual>
+    <collision>
+      <geometry><sphere radius="0.040"/></geometry>
     </collision>
     <inertial>
@@ -124,9 +129,9 @@
   <link name="caster_rear">
     <visual>
-      <geometry><sphere radius="0.045"/></geometry>
-      <material name="metallic_dark"/>
-    </visual>
-    <collision>
-      <geometry><sphere radius="0.045"/></geometry>
+      <geometry><sphere radius="0.040"/></geometry>
+      <material name="metallic_dark"/>
+    </visual>
+    <collision>
+      <geometry><sphere radius="0.040"/></geometry>
     </collision>
     <inertial>
@@ -190,4 +195,26 @@
     <origin xyz="0.05 0 1.15" rpy="0 0.35 0"/>
   </joint>
+  <!-- Contact properties: frictionless casters (they must slide, otherwise
+       they drag the robot and wheel odometry drifts), high-grip drive wheels -->
+  <gazebo reference="caster_front">
+    <mu1>0.0</mu1>
+    <mu2>0.0</mu2>
+  </gazebo>
+  <gazebo reference="caster_rear">
+    <mu1>0.0</mu1>
+    <mu2>0.0</mu2>
+  </gazebo>
+  <gazebo reference="left_wheel">
+    <mu1>1.0</mu1>
+    <mu2>1.0</mu2>
+    <kp>1000000.0</kp>
+    <kd>100.0</kd>
+  </gazebo>
+  <gazebo reference="right_wheel">
+    <mu1>1.0</mu1>
+    <mu2>1.0</mu2>
+    <kp>1000000.0</kp>
+    <kd>100.0</kd>
+  </gazebo>
   <!-- Gazebo Sim Differential Drive Plugin -->
   <gazebo>
